File: Eagle files/Project_design_v1.0.sch (EAGLE design)
At the start: 64 parts, among them CN1 USB_CONN, CN2 BATT_IN_JST, IC1 TPS73233DBVT, IC2 TPS73233DBVT, IC3 MCP73833T-AMI/MF, IC4 STM32F042K6T6, IC5 MCP9700T-E/TT, IC6 TLV379IDBVT, Q1 PMV16XN, Q2 PMV16XN, Q3 PMV16XN, Q4 PMV16XN

Commit message: schematic almose finished, part number edited, and PIR & buzzer added
Parts:
- removed C56, C58, C59, C60: 100n, custom_part:CAPA0402
- removed H1, H2, H3, H4: SOIL_MOISTURE, potentiometer:SOIL_MOISTURE
- removed IC4: STM32F042K6T6, stm32-microcontrollers:STM32F042K6T6
- removed IC5: MCP9700T-E/TT, MCP9700T-E_TT:MCP9700T-E/TT
- added C13, C14, C15, C16: 100n, custom_part:CAPA0402
- added C17, C18: 22pF, SparkFun:CAP0603-CAP
- added C20: 1uF, SparkFun:CAP0603-CAP
- added D5: Green, SparkFun:LED0603
- added D6: Yellow, SparkFun:LED0603
- added JP10, JP11, JP12, JP9: Connectors, pinhead:PINHD-1X2/90
- added JP13: PIN-1X3, pinhead:PINHD-1X3
- added JP7, JP8: M12PTH, SparkFun:M12PTH
- added LS1: BUZZER-PTH_KIT, SparkFun-Electromechanical:BUZZER-PTH_KIT
- added R13, R15, R16: 330, custom_part:0603RESIST
- added R14, R19, R21, R22: 10k, custom_part:0603RESIST
- added R17, R18: 22, SparkFun:RESISTOR0603-RES
- added U3: ATMEGA32U4, Testing:ATMEGA32U4OUTFAKES
- added Y1: 16MHz, SparkFun:CRYSTAL5X3
- JP1: value Contact_pin -> Connectors; device microbuilder:HEADER-1X2 -> pinhead:PINHD-1X2; PARTNO (none) -> /
- JP2, JP3, JP4, JP5, JP6: value Contact_pin -> Connectors; device microbuilder:HEADER-1X2 -> pinhead:PINHD-1X2/90
- R01, R02, R03: PARTNO ERJ-PA3F1002V -> ERJ-PA3F2001V
- R06, R07, R08: value 221 -> 330; PARTNO ERJ-PA3F2210V -> RC0603JR-07330RL
- R11, R12: value 221 -> 10k; PARTNO ERJ-PA3F2210V -> ERJ-PA3F1002V
Connections:
- removed net BOOT0: IC4.PB8/BOOT, R20.2
- removed net CHARGE_CMD: IC4.PA5/ADC_IN5
- removed net CTRL_MOIST1: H1.VCC
- removed net CTRL_MOIST2: H2.VCC
- removed net CTRL_MOIST3: H3.VCC
- removed net CTRL_MOIST4: H4.VCC
- removed net DAC_CLK: IC4.PA6/ADC_IN6
- removed net DAC_D2: IC4.PA7/ADC_IN7
- removed net DAC_D3: IC4.PA8
- removed net DAC_D4: IC4.PA9/USART1_TX
- removed net DAC_D5: IC4.PA10/USART1_RX
- removed net DAC_D6: IC4.PA11/USART1_CTS/CAN_RX
- removed net DAC_D7: IC4.PA12/USART1_CTS/CAN_TX
- removed net DAC_D8: IC4.PA15/USART2_RX
- removed net HV_DONE: IC4.PA4/ADC_IN4
- removed net LI_PRESET: IC4.PF0-OSC-IN
- removed net LOAD_CURRENT_1: IC4.PA0/USART2_CTS/ADC_IN0
- removed net LOAD_CURRENT_2: IC4.PA1/USART2_RTS/ADC_IN1
- removed net LOAD_CURRENT_3: IC4.PA2/USART2_TX/ADC_IN2
- removed net LOAD_CURRENT_4: IC4.PA3/USART2_RX/ADC_IN3
- removed net MUX_DIS: IC4.PB5
- removed net MUX_IN: IC4.PB0/ADC_IN8
- removed net MUX_S0: IC4.PB1/ADC_IN9
- removed net MUX_S1: IC4.PB3
- removed net MUX_S2: IC4.PB4
- removed net NRST: C59.1, IC4.NRST
- removed net SWCLK: IC4.PA14/SWCLK
- removed net SWDIO: IC4.PA13/SWDIO
- removed net TEMP_READ: IC5.VOUT
- removed net USART1_RX/I2C1_SDA: IC4.PB7/USART1_RX/I2C1_SDA
- removed net USART1_TX/I2C1_SCL: IC4.PB6/USART1_TX/I2C1_SCL
- new net A0: JP7.8, U3.PF7(ADC7)
- new net A1: JP7.7, U3.PF6(ADC6)
- new net A2: JP7.6, U3.PF5(ADC5)
- new net A3: JP7.5, U3.PF4(ADC4)
- new net A4: U3.PF1(ADC1)
- new net A5: U3.PF0(ADC0)
- new net ALARM: JP13.3
- new net AREF: U3.AREF
- new net BUZZ: LS1.1
- new net D+: R17.1, U3.D+
- new net D-: R18.1, U3.D-
- new net D10: JP7.12, U3.PB6(ADC13)
- new net D11: U3.PB7
- new net D12: U3.PD6(ADC9)
- new net D13: U3.PC7
- new net D14: U3.PB3(MISO)
- new net D2: JP8.8, U3.PD1(SDA)
- new net D3: JP8.7, U3.PD0(SCL)
- new net D4: JP8.6, U3.PD4(ADC8)
- new net D5: JP8.5, U3.PC6
- new net D6: JP8.4, U3.PD7(ADC10)
- new net D7: JP8.3, U3.PE6
- new net D8: JP8.2, U3.PB4(ADC11)
- new net D9: JP8.1, U3.PB5(ADC12)
- new net MISO: JP7.10, U3.PB0(SS)
- new net MOSI: JP7.11, U3.PB2(MOSI)
- new net N$18: C17.1, U3.XTAL1, Y1.2
- new net N$19: C20.2, U3.UCAP
- new net N$20: CN1.D-, R18.2
- new net N$21: CN1.D+, R17.2
- new net N$22: LS1.2, R13.1
- new net N$23: D6.C
- new net N$24: D5.C
- new net N$9: C18.1, U3.XTAL2, Y1.1
- new net RESET: JP7.3, U3.!RESET
- new net RXI: JP8.11, U3.PD2(RX)
- new net SCK: JP7.9, U3.PB1(SCK)
- new net TXLED: U3.PD5
- new net TXO: JP8.12, U3.PD3(TX)
- net 3.3V: now also JP13.1, R19.2, R20.2, R21.2, R22.2, U3.AVCC@24, U3.AVCC@44, U3.VCC@14, U3.VCC@34; no longer C10.1, C11.1, C56.1, C58.1, IC4.VDD, IC4.VDD-IO2, IC5.VDD
- net 5.0V: now also U3.UVCC, U3.VBUS
- net GND: now also C13.2, C15.2, C16.2, C17.2, C18.2, C20.1, JP10.2, JP11.2, JP12.2, JP13.2, JP7.1, JP7.2, JP8.10, JP8.9, JP9.2, R13.2, U3.GND@15, U3.GND@23, U3.GND@35, U3.GND@43, U3.PE2/!HWB, U3.UGND; no longer C10.2, C56.2, C58.2, C59.2, C60.2, H1.GND, H2.GND, H3.GND, H4.GND, IC4.VSS, IC4.VSS2, IC5.GND, R20.1
- net LED_G: no longer IC4.PF1-OSC-OUT
- net LEVEL_SENSOR: now also JP12.1; no longer JP6.1
- net MOISTURE1: now also C15.1, JP6.1, R19.1; no longer H1.VOUT
- net MOISTURE2: now also C11.1, JP9.1, R20.1; no longer H2.VOUT
- net MOISTURE3: now also C13.1, JP11.1, R21.1; no longer H3.VOUT
- net MOISTURE4: now also C16.1, JP10.1, R22.1; no longer H4.VOUT
- net VCC: now also D5.A, D6.A, JP7.4; no longer C60.1, IC4.VDDA
Other:
- note added: "Level sensor"
- note added: "Not used"
- note removed: "Bypassing Capacitor Analog + Digital"
- note removed: "Level Sensor"
- note removed: "Microcontroller"
- note removed: "TEMPERATURE SENSOR"
- note removed: "find a RGB LED with common cathode instead of common anode"
- moved on the sheet: C10, C11, JP2, JP6, R20

Commit message: schematics design uptaded and adjusted for exportation for the MS2
Connections:
- net 3.3V: now also C10.1, R14.2
- net GND: now also C10.2
- net RESET: now also R14.1
Other:
- note added: "DC-DC Converter: LDO"
- note added: "Microcontroller & connectors"
- note added: "PIR detector interface & buzzer"
- note removed: "DC-DC Converter"
- moved on the sheet: C1, C10, C12, C2, C3, C4, C5, C6, C7, C8, C9, CN1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

Commit message: PCB line + silkscreen updated
Parts:
- removed C10: 100n, custom_part:CAPA0402
- removed D5: Green, SparkFun:LED0603
- removed D6: Yellow, SparkFun:LED0603
- removed JP7, JP8: M12PTH, SparkFun:M12PTH
- removed U3: ATMEGA32U4, Testing:ATMEGA32U4OUTFAKES
- added D14/MISO, D16/MOSI: JUMPER-SMT_2_NO_SILK, SparkFun-Jumpers:JUMPER-SMT_2_NO_SILK
- added IC4: ATMEGA32U4, ATMEGA32U4:ATMEGA32U4TQFP-44
- added J1, J2: (no value), SparkFun-Connectors:CONN_01
- added J3: 455-1750-1-ND, SparkFun-Connectors:CONN_03
- added JP14, JP15: Connectors, SparkFun-Connectors:CONN_02
- added LD4: GRN, SparkFun-LED:LED3MM
- added LD5: RED, SparkFun-LED:LED3MM
- added Q5: PMV16XN, custom_part_2:PMV16XN
- added R23, R24, R25, R26, R30, R31: 10k, custom_part:0603RESIST
- added R27, R28, R29: 2k, custom_part:0603RESIST
- CN1: value USB_CONN -> WM9734TR-ND; device 105133-0011:105133-0011 -> SparkFun-Connectors:USB_MICRO-B_FEMALE-SMT-VERT; PARTNO 105133-0011 -> 1051330011
- H5: value SOIL_MOISTURE -> POT1
- H6: value SOIL_MOISTURE -> POT2
- H7: value SOIL_MOISTURE -> POT3
- H8: value SOIL_MOISTURE -> POT4
- IC3: value MCP73833T-AMI/MF -> MCP73833T-BZI/UN; device microbuilder:MCP73833DFN -> MCP73833T-BZI_UN:MCP73833T-BZI/UN; PARTNO MCP73833DFN -> (none)
- JP10, JP11, JP12, JP2, JP3, JP4, JP5, JP6, JP9: device pinhead:PINHD-1X2/90 -> SparkFun-Connectors:CONN_02; PARTNO (none) -> M20-9960245
- JP13: device pinhead:PINHD-1X3 -> pinhead:PINHD-2X2; PARTNO / -> M22-2040805
- LD1, LD2: value RGB_LED -> DIFFUSE; device Semicond:ASMB-MTB0-0A3A2PLCC-4 -> RGB_LED:LED_RGB_THRU_CA; CODE 2401105 -> (none); DISTRIBUTOR Farnell -> (none); LINK http://ch.farnell.com/fr-CH/broadcom-limited/asmb-mtb0-0a3a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 -> (none); PARTNO ASMB-MTB0-0A3A2 -> WP154A4SEJ3VBDZGW/CA; REFERENCE ASMB-MTB0-0A3A2 -> (none); UNIT_PRICE 0.332 -> (none)
- LD3: value RLED -> OR; device LTST-C190KRKT:LTST-C190KRKT -> SparkFun-LED:LED3MM; PARTNO LTST-C190KRKT -> TLHO4600
- R05, R10, R11, R12, R14, R19, R20, R21, R22: PARTNO ERJ-PA3F1002V -> ERA-3AEB103V
- R06, R07, R08: value 330 -> 1k
- R15, R16: value 330 -> 10k; PARTNO RC0603JR-07330RL -> ERA-3AEB103V
- Y1: value 16MHz -> 8MHz; PARTNO ABM3C-16.000MHZ-D4Y-T -> ABM3C-8.000MHZ-D4Y-T
- renumbered IC6 to IC5
Connections:
- removed net ALARM: JP13.3
- removed net BUZZ: LS1.1
- removed net CTRL_MOTOR1: Q1.G
- removed net CTRL_MOTOR2: Q2.G
- removed net CTRL_MOTOR3: Q3.G
- removed net CTRL_MOTOR4: Q4.G
- removed net CTRL_PHOTOCELL: R04.P$2
- removed net D10: JP7.12, U3.PB6(ADC13)
- removed net D11: U3.PB7
- removed net D12: U3.PD6(ADC9)
- removed net D13: U3.PC7
- removed net D14: U3.PB3(MISO)
- removed net D3: JP8.7, U3.PD0(SCL)
- removed net D4: JP8.6, U3.PD4(ADC8)
- removed net D5: JP8.5, U3.PC6
- removed net D6: JP8.4, U3.PD7(ADC10)
- removed net D9: JP8.1, U3.PB5(ADC12)
- removed net LED_B: R03.2
- removed net LED_G: R01.2
- removed net LED_R: R02.2
- removed net LEVEL_SENSOR: JP12.1
- removed net MISO: JP7.10, U3.PB0(SS)
- removed net MOISTURE1: C15.1, JP6.1, R19.1
- removed net MOISTURE2: C11.1, JP9.1, R20.1
- removed net MOISTURE3: C13.1, JP11.1, R21.1
- removed net MOISTURE4: C16.1, JP10.1, R22.1
- removed net MOSI: JP7.11, U3.PB2(MOSI)
- removed net N$23: D6.C
- removed net N$24: D5.C
- removed net PHOTOCELL_READ: R04.P$1, R05.2
- removed net RXI: JP8.11, U3.PD2(RX)
- removed net SCK: JP7.9, U3.PB1(SCK)
- removed net TXLED: U3.PD5
- removed net TXO: JP8.12, U3.PD3(TX)
- removed net V_BAT_SENSE: IC5.-IN, IC5.VOUT
- removed net WATER_ADJ_1: H5.VOUT
- removed net WATER_ADJ_2: H6.VOUT
- removed net WATER_ADJ_3: H7.VOUT
- removed net WATER_ADJ_4: H8.VOUT
- new net A10: C15.1, IC4.PD6(ADC9), JP6.1, R19.1
- new net A6: C13.1, IC4.PD4(ADC8), JP11.1, R21.1
- new net A7: C11.1, IC4.PD7(ADC10), JP9.1, R20.1
- new net A8: C16.1, IC4.PB5(ADC12), JP10.1, R22.1
- new net CTRL_3.3V: H5.VCC, H6.VCC, H7.VCC, H8.VCC, JP13.3, Q5.S, R04.P$2, R15.2, R19.2, R20.2, R21.2, R22.2
- new net D10#: IC4.PB6(ADC13), R01.2
- new net D11#: IC4.PB7, R28.2
- new net D13#: IC4.PC7, R02.2
- new net D14/MISO: D14/MISO.2, IC4.PB3(MISO), J2.1
- new net D15/SCK: IC4.PB1(SCK), JP12.1, R30.2, R31.1
- new net D16/MOSI: D16/MOSI.2, IC4.PB2(MOSI), J1.1
- new net D17/SS: IC4.PB0(SS), JP13.4
- new net D3#: IC4.PD0(SCL), LS1.1
- new net D5#: IC4.PC6, R03.2
- new net N$26: LD1.BLU, R29.1
- new net N$28: LD1.RED, R28.1
- new net N$29: LD1.GRN, R27.1
- new net N$30: D16/MOSI.1, R29.2
- new net N$32: D14/MISO.1, R27.2
- new net RXI/D0: IC4.PD2(RX), Q2.G, R25.2
- new net TXO/D1: IC4.PD3(TX), Q3.G, R23.2
- net 3.3V: now also IC4.AVCC@24, IC4.AVCC@44, IC4.VCC@14, IC4.VCC@34, J3.3, JP15.1, LD1.A, LD2.A, Q5.D, R31.2; no longer C10.1, H5.VCC, H6.VCC, H7.VCC, H8.VCC, JP13.1, LD1.1, R19.2, R20.2, R21.2, R22.2, U3.AVCC@24, U3.AVCC@44, U3.VCC@14, U3.VCC@34
- net 5.0V: now also IC3.VDD, IC3.VDD_2, IC4.UVCC, IC4.VBUS, LD4.A, LD5.A; no longer IC3.VDD1, IC3.VDD2, LD2.1, U3.UVCC, U3.VBUS
- net A0: now also H5.VOUT, IC4.PF7(ADC7); no longer JP7.8, U3.PF7(ADC7)
- net A1: now also H8.VOUT, IC4.PF6(ADC6); no longer JP7.7, U3.PF6(ADC6)
- net A2: now also H7.VOUT, IC4.PF5(ADC5); no longer JP7.6, U3.PF5(ADC5)
- net A3: now also H6.VOUT, IC4.PF4(ADC4); no longer JP7.5, U3.PF4(ADC4)
- net A4: now also IC4.PF1(ADC1), R04.P$1, R05.2; no longer U3.PF1(ADC1)
- net A5: now also IC4.PF0(ADC0), IC5.-IN, IC5.VOUT; no longer U3.PF0(ADC0)
- net AREF: now also C14.1, IC4.AREF; no longer U3.AREF
- net D+: now also IC4.D+; no longer U3.D+
- net D-: now also IC4.D-; no longer U3.D-
- net D2: now also IC4.PD1(SDA), Q1.G, R26.2; no longer JP8.8, U3.PD1(SDA)
- net D7: now also IC4.PE6, Q5.G, R16.2; no longer JP8.3, U3.PE6
- net D8: now also IC4.PB4(ADC11), Q4.G, R24.2; no longer JP8.2, U3.PB4(ADC11)
- net GND: now also C14.2, IC3.VSS, IC4.GND@15, IC4.GND@23, IC4.GND@35, IC4.GND@43, IC4.PE2/!HWB, IC4.UGND, J3.2, JP13.1, JP14.2, JP15.2, R15.1, R16.1, R23.1, R24.1, R25.1, R26.1, R30.1; no longer C10.2, IC3.GND, JP7.1, JP7.2, JP8.10, JP8.9, U3.GND@15, U3.GND@23, U3.GND@35, U3.GND@43, U3.PE2/!HWB, U3.UGND
- net N$1: now also LD2.GRN; no longer LD1.2
- net N$12: now also LD5.C; no longer LD3.C
- net N$18: now also IC4.XTAL1; no longer U3.XTAL1
- net N$19: now also IC4.UCAP; no longer U3.UCAP
- net N$3: now also LD3.C; no longer LD2.3
- net N$34: now also LD2.BLU; no longer LD1.3
- net N$35: now also LD2.RED; no longer LD1.4
- net N$4: now also LD4.C; no longer LD2.4
- net N$5: now also IC3.STAT2; no longer IC3.STAT1
- net N$6: now also IC3.STAT1; no longer IC3.STAT2
- net N$7: now also IC3.*PG; no longer IC3.PG
- net N$9: now also IC4.XTAL2; no longer U3.XTAL2
- net RESET: now also IC4.!RESET, J3.1; no longer JP7.3, U3.!RESET
- net VCC: now also JP14.1; no longer D5.A, D6.A, JP7.4
- net V_BAT: now also IC3.VBAT, IC3.VBAT_2; no longer IC3.VBAT1, IC3.VBAT2
Other:
- note removed: "ERJ-3EKF1002V"
- note removed: "Not used"
- note removed: "pwr"
- moved on the sheet: C14, C17, C18, C20, C7, C9, CN2, D1, D2, D3, D4, H5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
