File: Eagle files/Project_design_v1.0.sch (EAGLE design)
At the start: 96 parts, among them CN1 WM9734TR-ND, CN2 BATT_IN_JST, IC1 TPS73233DBVT, IC2 TPS73233DBVT, IC3 MCP73833T-BZI/UN, IC4 ATMEGA32U4, IC5 TLV379IDBVT, J3 455-1750-1-ND, Q1 PMV16XN, Q2 PMV16XN, Q3 PMV16XN, Q4 PMV16XN, Q5 PMV16XN, Y1 8MHz

Commit message: final version of the PCB, final BOM, and .gitignore file added; let's start coding
Other:
- moved on the sheet: R09
Changed lines of the file:
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@@
 <attribute name="PARTNO" x="-243.84" y="226.06" size="1.778" layer="96" rot="R90" display="off"/>
 </instance>
-<instance part="R09" gate="G$1" x="-236.22" y="210.82" rot="R90">
-<attribute name="PARTNO" x="-236.22" y="210.82" size="1.778" layer="96" rot="R90" display="off"/>
+<instance part="R09" gate="G$1" x="-236.22" y="208.28" rot="R90">
+<attribute name="PARTNO" x="-236.22" y="208.28" size="1.778" layer="96" rot="R90" display="off"/>
 </instance>
 <instance part="R10" gate="G$1" x="-251.46" y="208.28" rot="R90">
@@
 </segment>
 <segment>
-<wire x1="-236.22" y1="205.74" x2="-236.22" y2="198.12" width="0.1524" layer="91"/>
+<wire x1="-236.22" y1="203.2" x2="-236.22" y2="198.12" width="0.1524" layer="91"/>
 <pinref part="U$14" gate="G$1" pin="GND"/>
 <pinref part="R09" gate="G$1" pin="1"/>
@@
 <net name="N$16" class="0">
 <segment>
-<wire x1="-236.22" y1="220.98" x2="-236.22" y2="215.9" width="0.1524" layer="91"/>
+<wire x1="-236.22" y1="220.98" x2="-236.22" y2="213.36" width="0.1524" layer="91"/>
 <pinref part="R09" gate="G$1" pin="2"/>
 <pinref part="IC3" gate="A" pin="PROG"/>
