File: Eagle files/Project_design_v1.0.brd (EAGLE design)
At the start: 65 x 60 mm, 96 parts, among them CN1 WM9734TR-ND, CN2 BATT_IN_JST, IC1 TPS73233DBVT, IC2 TPS73233DBVT, IC3 MCP73833T-BZI/UN, IC4 ATMEGA32U4, IC5 TLV379IDBVT, J3 455-1750-1-ND, Q1 PMV16XN, Q2 PMV16XN, Q3 PMV16XN, Q4 PMV16XN, Q5 PMV16XN, Y1 8MHz

Commit message: final version of the PCB, final BOM, and .gitignore file added; let's start coding
Parts:
- moved R15 2.50 mm to (50.4, 42.3)
- moved H5 1.28 mm to (57.5, 20.5)
- moved H7 0.56 mm to (57.5, 28.5)
- moved H6 0.32 mm to (57.5, 32.5)
- moved CN2 0.28 mm to (12.5, 3.50)
- moved H8 0.24 mm to (57.5, 24.0)
- moved C20 0.10 mm to (40.0, 38.5)
Routing:
- net 3.3V: track 127.7 -> 94.0 mm
- net VCC: track 51.3 -> 70.9 mm
- net CTRL_3.3V: track 13.6 -> 17.7 mm
- net A4: track 82.2 -> 80.6 mm
- net 5.0V: track 35.4 -> 36.6 mm, vias 2 -> 3
- net A2: track 9.65 -> 9.09 mm
- net N$19: track 2.27 -> 2.81 mm
- net GND: vias 10 -> 32
- added copper zone on layer 1, net 3.3V
- added copper zone on layer 16, net 3.3V
- added copper zone on layer 16, net 5.0V
- added copper zone on layer 1, net VCC
Other:
- board text added: "POTENTIOMETER"
- board text added: "Project Design EPFL 11/2017-K.Sin #Team2 V1.0"
- board text added: "RGB LED"
- board text added: "USB CONN"
